File: hardware/dmxnow.kicad_sch (KiCad schematic)
At the start: 61 parts, among them J1 WAGO 2604-1103 (L N PE in), J2 DMX tail (1 GND 2 B 3 A), J3 PROG (3V3 GND D- D+ EN BOOT), J4 WAGO 2604-1103 (L_SW N PE out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, J5 WAGO 2604-1102 (VLED_IN GND_L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, J6 WAGO 2604-1105 (VLED CH1-CH4), J7 WAGO 2604-1103 (L_SW N PE out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, K1 G5RL-U1A-E DC5, Q1 AO3400A, Q2 AOD4184A, Q3 AOD4184A, Q4 AOD4184A, Q5 AOD4184A, SW1 PTS810 (BOOT/maintenance), U1 ESP32-C3-MINI-1-N4, U2 SP3485EN, U3 AP2112K-3.3, U4 74AHCT125

Commit message: hardware: générateur PCB, règles 230 V, CI KiCad 9, relecture
PE hors carte (arbitrage A9) : borniers 230 V en 2 pôles. Carte 146 x 54 mm.
Placement et routage 230 V/LED scriptés, routage signaux par Freerouting,
règles DRC d'isolement, contrôles de cohérence, sorties JLCPCB, workflow CI
KiCad 9 et liste de relecture humaine.

Co-Authored-By: Claude Opus 5.5 <noreply@anthropic.com>
Claude-Session: https://claude.ai/code/session_01B51M6ZY5abLxTmcevvc8Le
Parts:
- removed H4, H5: M3 NPTH, MountingHole:MountingHole_3.2mm_M3, symbol Mechanical:MountingHole
- H3: Section main -> strip
- J1: value WAGO 2604-1103 (L N PE in) -> WAGO 2604-1102 (L N in); footprint dmxnow:TerminalBlock_WAGO_2604-1103_1x03_P5.00mm_Horizontal -> dmxnow:TerminalBlock_WAGO_2604-1102_1x02_P5.00mm_Horizontal; symbol Connector:Screw_Terminal_01x03 -> Connector:Screw_Terminal_01x02; MPN 2604-1103 -> 2604-1102
- J2: footprint Connector_Wire:SolderWire-0.25sqmm_1x03_P4.2mm_D0.65mm_OD1.7mm_Relief -> Connector_Wire:SolderWire-0.25sqmm_1x03_P4.2mm_D0.65mm_OD1.7mm
- J4: value WAGO 2604-1103 (L_SW N PE out 1) -> WAGO 2604-1102 (L_SW N out 1); footprint dmxnow:TerminalBlock_WAGO_2604-1103_1x03_P5.00mm_Horizontal -> dmxnow:TerminalBlock_WAGO_2604-1102_1x02_P5.00mm_Horizontal; symbol Connector:Screw_Terminal_01x03 -> Connector:Screw_Terminal_01x02; MPN 2604-1103 -> 2604-1102
- J7: value WAGO 2604-1103 (L_SW N PE out 2, J4b) -> WAGO 2604-1102 (L_SW N out 2, J4b); footprint dmxnow:TerminalBlock_WAGO_2604-1103_1x03_P5.00mm_Horizontal -> dmxnow:TerminalBlock_WAGO_2604-1102_1x02_P5.00mm_Horizontal; symbol Connector:Screw_Terminal_01x03 -> Connector:Screw_Terminal_01x02; MPN 2604-1103 -> 2604-1102
Connections:
- removed net PE: J1.3 (Pin_3), J4.3 (Pin_3), J7.3 (Pin_3)
Other:
- moved on the sheet: D2, F1, K1, PS1, Q1, R5, R6, RV1
