File: hardware/dmxnow.kicad_sch (KiCad schematic)
At the start: 59 parts, among them J1 WAGO 2604-1102 (L N in), J2 DMX tail (1 GND 2 B 3 A), J3 PROG (3V3 GND D- D+ EN BOOT), J4 WAGO 2604-1102 (L_SW N out 1), J5 WAGO 2604-1102 (VLED_IN GND_L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, J6 WAGO 2604-1105 (VLED CH1-CH4), J7 WAGO 2604-1102 (L_SW N out 2,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, K1 G5RL-U1A-E DC5, Q1 AO3400A, Q2 AOD4184A, Q3 AOD4184A, Q4 AOD4184A, Q5 AOD4184A, SW1 PTS810 (BOOT/maintenance), U1 ESP32-C3-MINI-1-N4, U2 SP3485EN, U3 AP2112K-3.3, U4 74AHCT125

Commit message: hardware: PCB routé, passe de finition, sorties JLCPCB
Routage basse tension par Freerouting (session enregistrée dans
hardware/route/), passe de finition (mini-routeur A*, vias d'îlots,
nettoyage), contrôles : 0 liaison manquante, 0 violation au DRC local,
cohérence netlist/PCB/découpe. Pull-downs PWM côté principal, liaisons
0 ohm R20/R21 à la place des ponts de cuivre. Gerbers, perçages, V-cut,
BOM/CPL JLCPCB (base et option LED).

Co-Authored-By: Claude Opus 5.5 <noreply@anthropic.com>
Claude-Session: https://claude.ai/code/session_01B51M6ZY5abLxTmcevvc8Le
Parts:
- removed NT1: NetTie GND/GND_LED, NetTie:NetTie-2_SMD_Pad0.5mm, symbol Device:NetTie_2
- removed NT2: NetTie BOARD_SENSE/GND, NetTie:NetTie-2_SMD_Pad0.5mm, symbol Device:NetTie_2
- added R20: 0R, Resistor_SMD:R_0805_2012Metric, symbol Device:R
- added R21: 0R, Resistor_SMD:R_0603_1608Metric, symbol Device:R
- R15, R16, R17, R18: Section strip -> main
Connections:
- net BOARD_SENSE: now also R21.1
- net GND: now also R20.1, R21.2
- net GND_LED: now also R20.2
Other:
- moved on the sheet: H1, H2, H3, J6, Q2, Q3, Q4, Q5, R10, R11, R12, R13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

Commit message: hardware: relais G5RL-1A-E-HR, cotes WAGO 2604 et IRM-03 vérifiées sur fiches
- K1 : G5RL-U1A-E (bistable, incompatible avec la commande MOSFET) remplacé par
  G5RL-1A-E-HR DC5 (LCSC C113250), même implantation ; corps 29,0 x 12,7 mm.
- WAGO 2604 : rangées de broches à 8,2 mm (au lieu de 6), corps 16,3 mm + levier
  2,9 mm, largeur (n-1) x 5 + 7,4 mm, pastilles 1,9 x 2,8 mm.
- Placement : J1/J4/J7 décalés de 0,7 mm vers le bord (3 mm entre le bus N et les
  pastilles L_SW), J6 et canaux de 0,5 mm, H3 de 0,5 mm (chevauchement de courtyard).
- PS1 : empreinte KiCad IRM-03 conforme à la fiche Mean Well 2025-08-08.
- Références LCSC ajoutées (K1, WAGO 2604-1102, IRM-03-5).
- SPEC (4.5, V-HW-03/04/09/10), ADR 0005 amendé, REVIEW.md, index des fiches.

Co-Authored-By: Claude Opus 5.5 <noreply@anthropic.com>
Claude-Session: https://claude.ai/code/session_01B51M6ZY5abLxTmcevvc8Le
Parts:
- J1, J4, J5, J7: LCSC (none) -> C3309286
- K1: value G5RL-U1A-E DC5 -> G5RL-1A-E-HR DC5; footprint dmxnow:Relay_SPST_Omron_G5RL-U1A-E -> dmxnow:Relay_SPST_Omron_G5RL-1A-E-HR; LCSC (none) -> C113250; MPN Omron G5RL-U1A-E DC5 -> Omron G5RL-1A-E-HR DC5
- PS1: LCSC (none) -> C6969425
Changed lines of the file:
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@@
       )
     )
-    (property "LCSC" ""
+    (property "LCSC" "C3309286"
       (at 33.02 40.64 0)
       (id 5)
@@
       )
     )
-    (property "LCSC" ""
+    (property "LCSC" "C6969425"
       (at 124.46 43.18 0)
       (id 5)
@@
       )
     )
-    (property "Value" "G5RL-U1A-E DC5"
+    (property "Value" "G5RL-1A-E-HR DC5"
       (at 209.55 44.45 0)
       (id 1)
@@
       )
     )
-    (property "Footprint" "dmxnow:Relay_SPST_Omron_G5RL-U1A-E"
+    (property "Footprint" "dmxnow:Relay_SPST_Omron_G5RL-1A-E-HR"
       (at 209.55 46.99 0)
       (id 2)
@@
       )
     )
-    (property "MPN" "Omron G5RL-U1A-E DC5"
+    (property "MPN" "Omron G5RL-1A-E-HR DC5"
       (at 198.12 45.72 0)
       (id 4)
@@
       )
     )
-    (property "LCSC" ""
+    (property "LCSC" "C113250"
       (at 198.12 45.72 0)
       (id 5)
@@
       )
     )
-    (property "LCSC" ""
+    (property "LCSC" "C3309286"
       (at 241.3 40.64 0)
       (id 5)
@@
       )
     )
-    (property "LCSC" ""
+    (property "LCSC" "C3309286"
       (at 281.94 40.64 0)
       (id 5)
@@
       )
     )
-    (property "LCSC" ""
+    (property "LCSC" "C3309286"
       (at 38.1 243.84 0)
       (id 5)

Commit message: hardware: références LCSC complètes et vérifiées, estimation de coût
- Codes LCSC ajoutés pour toutes les pièces montées (U1, D1, U4, Q2-Q5, D3, SW1,
  F1, F2, RV1, C1, C7, C8, D4, J6) ; stock et prix relevés via l'API JLCPCB.
- F1 : Littelfuse 37405000410 (hors stock) remplacé par 37205000001 (C142835),
  même série TR5 372. U2 : MPN corrigé en SP3485EN-L/TR (C8963).
- WAGO 2604-1105 (J6) en rupture chez LCSC : noté dans la BOM.
- SPEC §6 : coût composants ≈ 33 $ à l'unité, ≈ 28 $ par nœud en série de 20.

Co-Authored-By: Claude Opus 5.5 <noreply@anthropic.com>
Claude-Session: https://claude.ai/code/session_01B51M6ZY5abLxTmcevvc8Le
Parts:
- C1: LCSC (none) -> C96123
- C7: LCSC (none) -> C88732; MPN (none) -> Rubycon 35YXJ470M10X16
- C8: LCSC (none) -> C1848
- D1: LCSC (none) -> C12067
- D3: LCSC (none) -> C113997
- D4: LCSC (none) -> C12624; MPN (none) -> KT-0603G
- F1: LCSC (none) -> C142835; MPN Littelfuse 37405000410 -> Littelfuse 37205000001
- F2: LCSC (none) -> C207061
- J6: LCSC (none) -> C3818651
- Q2, Q3, Q4, Q5: LCSC (none) -> C99124
- RV1: LCSC (none) -> C113236; MPN (none) -> 10D561K
- SW1: LCSC (none) -> C116501
- U1: LCSC (none) -> C2838502
- U2: MPN SP3485EEN-L/TR -> SP3485EN-L/TR
- U4: LCSC (none) -> C155176
Changed lines of the file:
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@@
       )
     )
-    (property "MPN" "Littelfuse 37405000410"
+    (property "MPN" "Littelfuse 37205000001"
       (at 63.5 43.18 0)
       (id 4)
@@
       )
     )
-    (property "LCSC" ""
+    (property "LCSC" "C142835"
       (at 63.5 43.18 0)
       (id 5)
@@
       )
     )
-    (property "MPN" ""
+    (property "MPN" "10D561K"
       (at 88.9 43.18 0)
       (id 4)
@@
       )
     )
-    (property "LCSC" ""
+    (property "LCSC" "C113236"
       (at 88.9 43.18 0)
       (id 5)
@@
       )
     )
-    (property "LCSC" ""
+    (property "LCSC" "C96123"
       (at 109.22 93.98 0)
       (id 5)
@@
       )
     )
-    (property "LCSC" ""
+    (property "LCSC" "C2838502"
       (at 213.36 119.38 0)
       (id 5)
@@
       )
     )
-    (property "LCSC" ""
+    (property "LCSC" "C116501"
       (at 398.78 91.44 0)
       (id 5)
@@
       )
     )
-    (property "MPN" ""
+    (property "MPN" "KT-0603G"
       (at 505.46 91.44 0)
       (id 4)
@@
       )
     )
-    (property "LCSC" ""
+    (property "LCSC" "C12624"
       (at 505.46 91.44 0)
       (id 5)
@@
       )
     )
-    (property "MPN" "SP3485EEN-L/TR"
+    (property "MPN" "SP3485EN-L/TR"
       (at 40.64 195.58 0)
       (id 4)
@@
       )
     )
-    (property "LCSC" ""
+    (property "LCSC" "C12067"
       (at 106.68 185.42 0)
       (id 5)
@@
       )
     )
-    (property "LCSC" ""
+    (property "LCSC" "C207061"
       (at 73.66 246.38 0)
       (id 5)
@@
       )
     )
-    (property "LCSC" ""
+    (property "LCSC" "C113997"
       (at 106.68 241.3 0)
       (id 5)
@@
       )
     )
-    (property "MPN" ""
+    (property "MPN" "Rubycon 35YXJ470M10X16"
       (at 139.7 246.38 0)
       (id 4)
@@
       )
     )
-    (property "LCSC" ""
+    (property "LCSC" "C88732"
       (at 139.7 246.38 0)
       (id 5)
@@
       )
     )
-    (property "LCSC" ""
+    (property "LCSC" "C1848"
       (at 170.18 246.38 0)
       (id 5)
@@
       )
     )
-    (property "LCSC" ""
+    (property "LCSC" "C155176"
       (at 203.2 248.92 0)
       (id 5)
@@
       )
     )
-    (property "LCSC" ""
+    (property "LCSC" "C155176"
       (at 241.3 248.92 0)
       (id 5)
@@
       )
     )
-    (property "LCSC" ""
+    (property "LCSC" "C155176"
       (at 279.4 248.92 0)
       (id 5)
@@
       )
     )
-    (property "LCSC" ""
+    (property "LCSC" "C155176"
       (at 314.96 248.92 0)
       (id 5)
@@
       )
     )
-    (property "LCSC" ""
+    (property "LCSC" "C155176"
       (at 350.52 254 0)
       (id 5)
@@
       )
     )
-    (property "LCSC" ""
+    (property "LCSC" "C99124"
       (at 93.98 309.88 0)
       (id 5)
@@
       )
     )
-    (property "LCSC" ""
+    (property "LCSC" "C99124"
       (at 185.42 309.88 0)
       (id 5)
@@
       )
     )
-    (property "LCSC" ""
+    (property "LCSC" "C99124"
       (at 276.86 309.88 0)
       (id 5)
@@
       )
     )
-    (property "LCSC" ""
+    (property "LCSC" "C99124"
       (at 368.3 309.88 0)
       (id 5)
@@
       )
     )
-    (property "LCSC" ""
+    (property "LCSC" "C3818651"
       (at 403.86 309.88 0)
       (id 5)

Commit message: hardware: rév. 0.3 après revue de conception (3 relecteurs indépendants)
Bloquants corrigés :
- V-cut remplacé par une fente fraisée + 3 languettes perforées : la rainure
  V aurait coupé en fabrication les 7 pistes qui traversent la découpe, et
  JLCPCB refuse le V-cut sous 70 x 70 mm (ADR 0007 amendé).
- Fichiers de placement convertis aux conventions JLCPCB (SOT-23, SOT-23-5,
  SOIC, TO-252, ESP32-C3-MINI-1, centres des traversants) ; variantes BOM/CPL
  « full » (CMS + traversants) et « smt ».
- F1 : fusible céramique 5x20 T500mA H (1500 A) dans un support Schurter
  0031.8201, placé dans une bande de 10 mm ajoutée au-dessus de la zone 230 V.
- R15-R18 4,7k : GPIO6 (PWM1) a un pull-up interne ~45k au reset, le canal 1
  s'allumait au démarrage.

Autres corrections :
- Vias 0,9/0,35 mm (anneau >= 0,254 mm exigé en 2 oz), perçage WAGO 1,4 mm.
- Aucun via dans une pastille CMS (Freerouting via_at_smd off, routeur de
  finition, nouveau contrôle dans check.py).
- MOSFET AOD2610E 60 V (R-10 clos), C7 Nichicon UHW 2 A d'ondulation.
- Cuivre 230 V élargi (bus N 7,1 mm, doigts L_SW 7,4 mm), 3 vias par source.
- R22 pull-up DMX_TX, C10 47 uF sur +5V, R23 pull-up BOARD_SENSE, R19 100R.
- Zone interdite de 7,2 mm autour de la broche NC de PS1 (rangée AC).
- Règle DRC d'exception limitée aux pastilles de K1 et PS1.
- Plans LED avec pastilles traversantes en réserves thermiques, marquage
  de polarité de J5, via de masse pré-placés sur les pastilles isolées.
- SPEC, REVIEW.md et README mis à jour.

Co-Authored-By: Claude Opus 5.5 <noreply@anthropic.com>
Claude-Session: https://claude.ai/code/session_01B51M6ZY5abLxTmcevvc8Le
Parts:
- added C10: 47uF 10V, Capacitor_SMD:C_1206_3216Metric, symbol Device:C
- added R22: 10k, Resistor_SMD:R_0603_1608Metric, symbol Device:R
- added R23: 100k, Resistor_SMD:R_0603_1608Metric, symbol Device:R
- C4, C5, C6: value 1uF 16V -> 1uF
- C7: LCSC C88732 -> C136284; MPN Rubycon 35YXJ470M10X16 -> Nichicon UHW1V471MPD
- F1: value TR5 T500mA 250V -> 5x20 holder, T500mA H; footprint Fuse:Fuse_Littelfuse_372_D8.50mm -> Fuse:Fuseholder_Cylinder-5x20mm_Schurter_0031_8201_Horizontal_Open; LCSC C142835 -> C3204125; MPN Littelfuse 37205000001 -> Schurter 0031.8201
- Q2, Q3, Q4, Q5: value AOD4184A -> AOD2610E; LCSC C99124 -> C282428; MPN AOD4184A -> AOD2610E
- R15, R16, R17, R18: value 100k -> 4.7k; LCSC C25803 -> C23162
- R19: value 1k -> 100R; LCSC C21190 -> C22775
Connections:
- net +3V3: now also R22.1, R23.1
- net +5V: now also C10.1
- net BOARD_SENSE: now also R23.2
- net DMX_TX: now also R22.2
- net GND: now also C10.2
Other:
- moved on the sheet: C1, C2, C3, C4, C6, C7, C8, C9, D1, D2, D3, D4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

Commit message: hardware: troisième passe de revue (RV1, canari KiCad 9, centre K1)
- RV1 : empreinte du projet, perçage 1,1 mm (pattes 0,8 +-0,1 mm, le 0,8 mm
  de KiCad était trop juste avec la tolérance JLCPCB) et corps jusqu'à 9 mm
  d'épaisseur (fiche HEL 10D) ; RV1 décalé à X = 28,5, bus L_SW raccourci.
- drc_canary.py : constante d'unités renommée dans KiCad 9 (échec CI).
- CPL : centre de K1 = centre des broches (empreinte JLC).
- REVIEW.md : RV1, découplage 3V3 et pistes d'alimentation à 0,2 mm,
  découpage du plan de masse en face arrière (points de la 3e passe).

Contrôles locaux : netlist 0 erreur, PCB 0 erreur, DRC 0 erreur /
0 non connecté, canari OK.

Co-Authored-By: Claude Opus 5.5 <noreply@anthropic.com>
Claude-Session: https://claude.ai/code/session_01B51M6ZY5abLxTmcevvc8Le
Parts:
- RV1: footprint Varistor:RV_Disc_D12mm_W4.2mm_P7.5mm -> dmxnow:RV_Disc_D12mm_T9mm_P7.5mm_Drill1.1
Changed lines of the file:
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@@
       )
     )
-    (property "Footprint" "Varistor:RV_Disc_D12mm_W4.2mm_P7.5mm"
+    (property "Footprint" "dmxnow:RV_Disc_D12mm_T9mm_P7.5mm_Drill1.1"
       (at 92.202 43.18 90)
       (id 2)

Commit message: hardware: quatrième passe de revue (PS1, RV1, J6, fentes, marquages)
- PS1 : empreinte du projet, perçages 1,0 mm (broches 0,6 +-0,1 mm).
- RV1 : classé traversant (il figurait dans la BOM CMS), centre CPL entre
  les pattes.
- J6 (0 stock JLCPCB) retiré des fichiers d'assemblage JLCPCB, signalé dans
  bom_full.csv.
- Fentes d'isolement 1,2 mm à bouts arrondis ; bande F1 portée à 11,5 mm
  (support de 10,8 mm) ; traits de sérigraphie >= 0,15 mm.
- Marquages : IN/OUT L/N sur J1/J4/J7, GND B- A+ sur J2, V+ 1-4 sur J6.
- REVIEW.md §7 (commande et montage), SPEC : charge rubans <= 16 A.

Contrôles : netlist 0, PCB 0, DRC 0 erreur / 0 non connecté, canari OK.

Co-Authored-By: Claude Opus 5.5 <noreply@anthropic.com>
Claude-Session: https://claude.ai/code/session_01B51M6ZY5abLxTmcevvc8Le
Parts:
- PS1: footprint Converter_ACDC:Converter_ACDC_MeanWell_IRM-03-xx_THT -> dmxnow:Converter_ACDC_MeanWell_IRM-03-xx_THT_Drill1.0
Changed lines of the file:
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@@
       )
     )
-    (property "Footprint" "Converter_ACDC:Converter_ACDC_MeanWell_IRM-03-xx_THT"
+    (property "Footprint" "dmxnow:Converter_ACDC_MeanWell_IRM-03-xx_THT_Drill1.0"
       (at 127 52.07 0)
       (id 2)
